Commit message: Basic Gazebo Install

File: ora_description/description/dimensions.xacro (robot description, xacro)
@@ -32,7 +32,7 @@
   <xacro:property name="lidar_radius" value="${lidar_diameter / 2}"/>
   <xacro:property name="lidar_height" value="${0.051}"/>
-  <xacro:property name="lidar_z_offset" value="${(base_height / 2) + lidar_radius}"/>
+  <xacro:property name="lidar_z_offset" value="${base_height + 0.02}"/>
   <xacro:property name="lidar_y_offset" value="${0.0}"/>
-  <xacro:property name="lidar_x_offset" value="${0.0}"/>
+  <xacro:property name="lidar_x_offset" value="${(3 * base_length) / 4}"/>
   <!-- Zed -->
   <xacro:arg name="camera_name"   default="zed" />

File: ora_description/description/robot.urdf.xacro (robot description, xacro)
@@ -3,3 +3,6 @@
   <!-- Include all of the pieces of the robot -->
   <xacro:include filename="robot_core.xacro"/>
+  <xacro:include filename="gazebo_control.xacro"/>
+  <!-- Sensors -->
+  <xacro:include filename="lidar.xacro"/>
 </robot>

File: ora_description/description/robot_core.xacro (robot description, xacro)
@@ -34,4 +34,7 @@
     </xacro:inertial_box>
   </link>
+  <gazebo reference="chassis_link">
+    <material>Gazebo/White</material>
+  </gazebo>
   <!-- WHEELS -->
   <!-- LEFT WHEEL LINK -->
@@ -58,4 +61,7 @@
     </xacro:inertial_cylinder>
   </link>
+  <gazebo reference="left_wheel_link">
+    <material>Gazebo/Black</material>
+  </gazebo>
   <!-- RIGHT WHEEL LINK -->
   <joint name="right_wheel_joint" type="continuous">
@@ -81,4 +87,7 @@
     </xacro:inertial_cylinder>
   </link>
+  <gazebo reference="right_wheel_link">
+    <material>Gazebo/Black</material>
+  </gazebo>
   <!-- CASTER WHEEL LINK -->
   <joint name="caster_joint" type="fixed">
@@ -104,3 +113,10 @@
     </xacro:inertial_sphere>
   </link>
+  <gazebo reference="caster_wheel_link">
+      <material>Gazebo/Black</material>
+      <!-- Frictionless-ish -->
+      <!-- Stops the robot from jumping around -->
+      <mu1 value="0.001"/>
+      <mu2 value="0.001"/>
+    </gazebo>
 </robot>

Commit message: Added GPS to URDF

File: ora_description/description/dimensions.xacro (robot description, xacro)
@@ -35,4 +35,11 @@
   <xacro:property name="lidar_y_offset" value="${0.0}"/>
   <xacro:property name="lidar_x_offset" value="${(3 * base_length) / 4}"/>
+  <!-- GPS -->
+  <xacro:property name="gps_diameter" value="${0.035}"/>
+  <xacro:property name="gps_radius" value="${gps_diameter / 2}"/>
+  <xacro:property name="gps_height" value="${0.02}"/>
+  <xacro:property name="gps_z_offset" value="${base_height + 0.02}"/>
+  <xacro:property name="gps_y_offset" value="${0.0}"/>
+  <xacro:property name="gps_x_offset" value="${0.0}"/>
   <!-- Zed -->
   <xacro:arg name="camera_name"   default="zed" />

Commit message: fix GPS URDF

File: ora_description/description/dimensions.xacro (robot description, xacro)
@@ -39,7 +39,7 @@
   <xacro:property name="gps_radius" value="${gps_diameter / 2}"/>
   <xacro:property name="gps_height" value="${0.02}"/>
-  <xacro:property name="gps_z_offset" value="${base_height + 0.02}"/>
+  <xacro:property name="gps_z_offset" value="${base_height}"/>
   <xacro:property name="gps_y_offset" value="${0.0}"/>
-  <xacro:property name="gps_x_offset" value="${0.0}"/>
+  <xacro:property name="gps_x_offset" value="${base_length / 2}"/>
   <!-- Zed -->
   <xacro:arg name="camera_name"   default="zed" />

File: ora_description/description/gps.xacro (robot description, xacro)
@@ -1,34 +1,51 @@
 <?xml version="1.0"?>
 <robot xmlns:xacro="https://www.ros.org/wiki/xacro">
-  <joint name="base_joint" type="fixed">
+  <joint name="gps_joint" type="fixed">
     <parent link="base_link"/>
-    <child link="base_footprint" />
+    <child link="gps_link" />
     <origin xyz="${gps_x_offset} ${gps_y_offset} ${gps_z_offset}" rpy="0 0 0"/>
   </joint>
-  <sensor name="tb3_gps" type="gps">
-    <always_on>true</always_on>
-    <update_rate>1</update_rate>
-    <pose>0 0 0 0 0 0</pose>
-    <gps>
-      <position_sensing>
-        <horizontal>
-          <noise type="gaussian">
-            <mean>0.0</mean>
-            <stddev>0.01</stddev>
-          </noise>
-        </horizontal>
-        <vertical>
-          <noise type="gaussian">
-            <mean>0.0</mean>
-            <stddev>0.01</stddev>
-          </noise>
-        </vertical>
-      </position_sensing>
-    </gps>
-    <plugin name="gps_controller" filename="libgazebo_ros_gps_sensor.so">
-      <ros>
-        <remapping>~/out:=/gps/fix</remapping>
-      </ros>
-    </plugin>
-  </sensor>
+  <link name="gps_link">
+    <visual>
+      <geometry>
+        <cylinder radius="${gps_radius}" length="${gps_height}" />
+      </geometry>
+    </visual>
+    <collision>
+      <geometry>
+        <cylinder radius="${gps_radius}" length="${gps_height}" />
+      </geometry>
+    </collision>
+    <xacro:inertial_cylinder mass="0.15" length="${gps_height}" radius="${gps_radius}">
+      <origin xyz="0 0 0" rpy="0 0 0"/>
+    </xacro:inertial_cylinder>
+  </link>
+  <gazebo>
+    <sensor name="tb3_gps" type="gps">
+      <always_on>true</always_on>
+      <update_rate>1</update_rate>
+      <pose>0 0 0 0 0 0</pose>
+      <gps>
+        <position_sensing>
+          <horizontal>
+            <noise type="gaussian">
+              <mean>0.0</mean>
+              <stddev>0.01</stddev>
+            </noise>
+          </horizontal>
+          <vertical>
+            <noise type="gaussian">
+              <mean>0.0</mean>
+              <stddev>0.01</stddev>
+            </noise>
+          </vertical>
+        </position_sensing>
+      </gps>
+      <plugin name="gps_controller" filename="libgazebo_ros_gps_sensor.so">
+        <ros>
+          <remapping>~/out:=/gps/fix</remapping>
+        </ros>
+      </plugin>
+    </sensor>
+  </gazebo>
 </robot>

File: ora_description/description/robot.urdf.xacro (robot description, xacro)
@@ -23,3 +23,4 @@
   <xacro:include filename="lidar.xacro"/>
   <!-- <xacro:include filename="camera.xacro"/> -->
+  <xacro:include filename="gps.xacro" />
 </robot>

Commit message: fix URDF dimensions

File: ora_description/description/dimensions.xacro (robot description, xacro)
@@ -8,7 +8,8 @@
   <xacro:property name="in_to_m" value="${0.0254}"/>
   <!-- Base Chassis Dimensions -->
-  <xacro:property name="base_length" value="${0.508}"/>
-  <xacro:property name="base_width" value="${0.406}"/>
-  <xacro:property name="base_height" value="${0.406}"/>
+  <xacro:property name="chassis_offset" value="${(base_length / 2) - wheel_x_center_to_back - (wheel_radius / 1.5)}" />
+  <xacro:property name="base_length" value="${0.914}"/>
+  <xacro:property name="base_width" value="${0.508}"/>
+  <xacro:property name="base_height" value="${0.508}"/>
   <!-- Wheel Dimensions / Location -->
   <xacro:property name="wheel_diameter" value="${203.101 * mm_to_m}"/>
@@ -19,5 +20,5 @@
   <xacro:property name="wheel_y_offset" value="${(base_width / 2) + 2 * wheel_y_gap}"/>
   <xacro:property name="wheel_x_center_to_back" value="${.095}"/>
-  <xacro:property name="wheel_x_offset" value="${(base_length / 2) - wheel_x_center_to_back - (wheel_radius / 1.5)}"/>
+  <xacro:property name="wheel_x_offset" value="${chassis_offset + (wheel_radius / 2)}"/>
   <!-- Caster Dimensions / Location -->
   <xacro:property name="caster_diameter" value="${0.052}"/>
@@ -32,5 +33,5 @@
   <xacro:property name="lidar_radius" value="${lidar_diameter / 2}"/>
   <xacro:property name="lidar_height" value="${0.051}"/>
-  <xacro:property name="lidar_z_offset" value="${base_height + 0.02}"/>
+  <xacro:property name="lidar_z_offset" value="${base_height + 0.04}"/>
   <xacro:property name="lidar_y_offset" value="${0.0}"/>
   <xacro:property name="lidar_x_offset" value="${(3 * base_length) / 4}"/>

File: ora_description/description/lidar.xacro (robot description, xacro)
@@ -48,5 +48,5 @@
         <range>
           <!-- 0.15-12.0 per the datasheet -->
-          <min>0.3</min>
+          <min>0.35</min>
           <max>12.0</max>
           <resolution>0.01</resolution>

File: ora_description/description/robot_core.xacro (robot description, xacro)
@@ -20,5 +20,5 @@
     <parent link="base_link"/>
     <child link="chassis_link"/>
-    <origin xyz="${wheel_x_offset} 0 0" rpy="0 0 0"/>
+    <origin xyz="${chassis_offset} 0 0" rpy="0 0 0"/>
   </joint>
   <link name="chassis_link">
@@ -100,5 +100,5 @@
     <parent link="chassis_link"/>
     <child link="caster_wheel_link"/>
-    <origin xyz="-${caster_x_offset} ${caster_y_offset} ${caster_z_offset}" rpy="0 0 0"/>
+    <origin xyz="${caster_x_offset} ${caster_y_offset} ${caster_z_offset}" rpy="0 0 0"/>
     <axis xyz="0 0 1"/>
   </joint>

Commit message: Fixed the robot description

File: ora_description/description/dimensions.xacro (robot description, xacro)
@@ -20,5 +20,5 @@
   <xacro:property name="wheel_y_offset" value="${(base_width / 2) + 2 * wheel_y_gap}"/>
   <xacro:property name="wheel_x_center_to_back" value="${.095}"/>
-  <xacro:property name="wheel_x_offset" value="${chassis_offset + (wheel_radius / 2)}"/>
+  <xacro:property name="wheel_x_offset" value="${(wheel_radius / 2)}"/>
   <!-- Caster Dimensions / Location -->
   <xacro:property name="caster_diameter" value="${0.052}"/>
@@ -28,5 +28,5 @@
   <xacro:property name="caster_y_offset" value="${0}"/>
   <xacro:property name="caster_x_front_to_caster" value="${0.0905}"/>
-  <xacro:property name="caster_x_offset" value="${base_length - caster_x_front_to_caster}"/>
+  <xacro:property name="caster_x_offset" value="${base_length - caster_x_front_to_caster - (10 * in_to_m)}"/>
   <!-- Lidar -->
   <xacro:property name="lidar_diameter" value="${0.070}"/>
@@ -35,5 +35,5 @@
   <xacro:property name="lidar_z_offset" value="${base_height + 0.04}"/>
   <xacro:property name="lidar_y_offset" value="${0.0}"/>
-  <xacro:property name="lidar_x_offset" value="${(3 * base_length) / 4}"/>
+  <xacro:property name="lidar_x_offset" value="${4 * in_to_m}"/>
   <!-- GPS -->
   <xacro:property name="gps_diameter" value="${0.035}"/>
@@ -42,5 +42,5 @@
   <xacro:property name="gps_z_offset" value="${base_height}"/>
   <xacro:property name="gps_y_offset" value="${0.0}"/>
-  <xacro:property name="gps_x_offset" value="${base_length / 2}"/>
+  <xacro:property name="gps_x_offset" value="${11.5 * in_to_m}"/>
   <!-- Zed -->
   <xacro:arg name="camera_name"   default="zed" />
@@ -49,4 +49,4 @@
   <xacro:property name="zed_z_offset" value="${0.508}"/>
   <xacro:property name="zed_y_offset" value="${0.0}"/>
-  <xacro:property name="zed_x_offset" value="${base_length / 2}"/>
+  <xacro:property name="zed_x_offset" value="${8.5 * in_to_m}"/>
 </robot>

File: ora_description/description/robot_core.xacro (robot description, xacro)
@@ -20,5 +20,5 @@
     <parent link="base_link"/>
     <child link="chassis_link"/>
-    <origin xyz="${chassis_offset} 0 0" rpy="0 0 0"/>
+    <origin xyz="0 0 0" rpy="0 0 0"/>
   </joint>
   <link name="chassis_link">

File: ora_description/description/ros2_control.xacro (robot description, xacro)
@@ -9,8 +9,8 @@
       <hardware>
         <plugin>odrive_ros2_control_plugin/ODriveHardwareInterface</plugin>
-        <param name="can">can0</param>
+        <param name="can">can1</param>
       </hardware>
       <joint name="left_wheel_joint">
-        <param name="node_id">1</param>
+        <param name="node_id">0</param>
         <param name="invert">true</param>
         <command_interface name="velocity"/>
@@ -20,5 +20,5 @@
       </joint>
       <joint name="right_wheel_joint">
-        <param name="node_id">0</param>
+        <param name="node_id">1</param>
         <param name="invert">false</param>
         <command_interface name="velocity"/>
