Commit message: ros2 control config

File: ora_description/description/camera.xacro (robot description, xacro)
@@ -1,13 +1,19 @@
 <?xml version="1.0"?>
 <robot xmlns:xacro="https://www.ros.org/wiki/xacro">
-  <!-- <xacro:include filename="$(find zed_wrapper)/urdf/zed_macro.urdf.xacro"/> -->
-  <!-- <xacro:zed_camera name="$(arg camera_name)" model="$(arg camera_model)" enable_gnss="false">
-    <gnss_origin xyz="0 0 0" rpy="0 0 0"/>
-  </xacro:zed_camera>-->
+  <!-- Get the ZED description -->
+  <xacro:include filename="$(find zed_wrapper)/urdf/zed_macro.urdf.xacro"/>
+  <!-- Make the camera -->
+  <!-- Either using GNSS or not -->
+  <xacro:zed_camera name="$(arg camera_name)" model="$(arg camera_model)" enable_gnss="$(use_zed_localization)">
+    <xacro:if value="$(use_zed_localization)">
+      <gnss_origin xyz="0 0 0" rpy="0 0 0"/>
+    </xacro:if>
+  </xacro:zed_camera>
   <!-- Add a joint to connect the ZED Camera to the robot -->
-  <!-- <joint name="$(arg camera_name)_joint" type="fixed">
+  <joint name="$(arg camera_name)_joint" type="fixed">
+  <!-- '$(arg camera_name)_camera_link' is a child of 'base_link' -->
     <parent link="base_link"/>
     <child link="$(arg camera_name)_camera_link"/>
-    <origin xyz="${zed_x_offset} 0 ${zed_z_offset}" rpy="0 ${40 * (pi / 180)} 0" />
-  </joint> -->
+    <origin xyz="${zed_x_offset} 0 ${zed_z_offset}" rpy="0 0 0" />
+  </joint>
 </robot>

File: ora_description/description/robot.urdf.xacro (robot description, xacro)
@@ -2,6 +2,13 @@
 <robot xmlns:xacro="https://www.ros.org/wiki/xacro" name="robot_name">
   <!-- Args -->
+  <!-- General -->
+  <xacro:arg name="sim_mode" default="false"/>
+  <!-- ROS2 control -->
   <xacro:arg name="use_ros2_control" default="true"/>
-  <xacro:arg name="sim_mode" default="false"/>
+  <!-- Zed -->
+  <xacro:arg name="camera_name" default="zed"/>
+  <xacro:arg name="camera_model" default="zed2i"/>
+  <xacro:arg name="use_zed_localization" default="true" />
+  <xacro:arg name="baseline" default="0.0" />
   <!-- Include all of the pieces of the robot -->
   <xacro:include filename="robot_core.xacro"/>
@@ -15,4 +22,4 @@
   <!-- Sensors -->
   <xacro:include filename="lidar.xacro"/>
-  <xacro:include filename="camera.xacro"/>
+  <!-- <xacro:include filename="camera.xacro"/> -->
 </robot>

File: ora_description/description/ros2_control.xacro (robot description, xacro)
@@ -6,27 +6,28 @@
   <xacro:unless value="$(arg sim_mode)">
     <ros2_control name="RealRobot" type="system">
+      <!-- ODrive ros2 control package -->
       <hardware>
-        <!-- Custom plugin made for the ODrive S1s -->
-        <!-- Please dont ask me about this, it was painful to make -->
-        <plugin>gazebo_ros2_control/GazeboSystem</plugin>
+        <plugin>odrive_ros2_control_plugin/ODriveHardwareInterface</plugin>
+        <param name="can">can0</param>
       </hardware>
       <joint name="left_wheel_joint">
-        <command_interface name="velocity">
-          <param name="min">-10</param>
-          <param name="max">10</param>
-        </command_interface>
+        <param name="node_id">1</param>
+        <param name="invert">true</param>
+        <command_interface name="velocity"/>
         <state_interface name="velocity"/>
         <state_interface name="position"/>
+        <state_interface name="effort"/>
       </joint>
       <joint name="right_wheel_joint">
-        <command_interface name="velocity">
-          <param name="min">-10</param>
-          <param name="max">10</param>
-        </command_interface>
+        <param name="node_id">0</param>
+        <param name="invert">false</param>
+        <command_interface name="velocity"/>
         <state_interface name="velocity"/>
         <state_interface name="position"/>
+        <state_interface name="effort"/>
       </joint>
     </ros2_control>
   </xacro:unless>
+  <!-- Real Robot Config -->
   <!-- Simulated Robot Config -->
   <xacro:if value="$(arg sim_mode)">
@@ -59,3 +60,4 @@
     </gazebo>
   </xacro:if>
+  <!-- Simulated Robot Config -->
 </robot>

Commit message: Joint Fixes

File: ora_description/description/camera.xacro (robot description, xacro)
@@ -15,5 +15,5 @@
     <parent link="base_link"/>
     <child link="$(arg camera_name)_camera_link"/>
-    <origin xyz="${zed_x_offset} 0 ${zed_z_offset}" rpy="0 0 0" />
+    <origin xyz="${-zed_x_offset} 0 ${zed_z_offset}" rpy="0 ${20 * (pi / 180)} 0" />
   </joint>
 </robot>

File: ora_description/description/dimensions.xacro (robot description, xacro)
@@ -47,5 +47,5 @@
   <xacro:arg name="camera_model"  default="zed2i" />
   <xacro:arg name="use_zed_localization" default="true" />
-  <xacro:property name="zed_z_offset" value="${0.508}"/>
+  <xacro:property name="zed_z_offset" value="${0.508 + (8.75 * in_to_m)}"/>
   <xacro:property name="zed_y_offset" value="${0.0}"/>
   <xacro:property name="zed_x_offset" value="${8.5 * in_to_m}"/>

File: ora_description/description/gps.xacro (robot description, xacro)
@@ -4,5 +4,5 @@
     <parent link="base_link"/>
     <child link="gps_link" />
-    <origin xyz="${gps_x_offset} ${gps_y_offset} ${gps_z_offset}" rpy="0 0 0"/>
+    <origin xyz="${-gps_x_offset} ${gps_y_offset} ${gps_z_offset}" rpy="0 0 0"/>
   </joint>
   <link name="gps_link">

File: ora_description/description/lidar.xacro (robot description, xacro)
@@ -6,5 +6,5 @@
     <parent link="chassis_link"/>
     <child link="laser_frame"/>
-    <origin xyz="${lidar_x_offset} ${lidar_y_offset} ${lidar_z_offset}" rpy="0 0 0"/>
+    <origin xyz="${-lidar_x_offset} ${lidar_y_offset} ${lidar_z_offset}" rpy="0 0 ${pi}"/>
   </joint>
   <!-- Laser frame follows some  -->

File: ora_description/description/robot_core.xacro (robot description, xacro)
@@ -24,5 +24,5 @@
   <link name="chassis_link">
     <visual>
-      <origin xyz="${base_length / 2} 0 ${base_height / 2}" rpy="0 0 0"/>
+      <origin xyz="${-base_length / 2} 0 ${base_height / 2}" rpy="0 0 0"/>
       <geometry>
         <box size="${base_length} ${base_width} ${base_height}"/>
@@ -31,5 +31,5 @@
     </visual>
     <collision>
-      <origin xyz="${base_length / 2} 0 ${base_height / 2}" rpy="0 0 0"/>
+      <origin xyz="${-base_length / 2} 0 ${base_height / 2}" rpy="0 0 0"/>
       <geometry>
         <box size="${base_length} ${base_width} ${base_height}"/>
@@ -37,5 +37,5 @@
     </collision>
     <xacro:inertial_box mass="10.0" x="${base_length}" y="${base_width}" z="${base_height}">
-      <origin xyz="${base_length / 2} 0 ${base_height / 2}" rpy="0 0 0"/>
+      <origin xyz="${-base_length / 2} 0 ${base_height / 2}" rpy="0 0 0"/>
     </xacro:inertial_box>
   </link>
@@ -48,5 +48,5 @@
     <parent link="base_link"/>
     <child link="left_wheel_link"/>
-    <origin xyz="${wheel_x_offset} ${wheel_y_offset} ${wheel_z_offset}" rpy="-${pi / 2} 0.0 0.0"/>
+    <origin xyz="${-wheel_x_offset} ${wheel_y_offset} ${wheel_z_offset}" rpy="-${pi / 2} 0.0 0.0"/>
     <axis xyz="0 0 -1"/>
   </joint>
@@ -74,5 +74,5 @@
     <parent link="base_link"/>
     <child link="right_wheel_link"/>
-    <origin xyz="${wheel_x_offset} -${wheel_y_offset} ${wheel_z_offset}" rpy="${pi / 2} 0.0 0.0"/>
+    <origin xyz="${-wheel_x_offset} -${wheel_y_offset} ${wheel_z_offset}" rpy="${pi / 2} 0.0 0.0"/>
     <axis xyz="0 0 1"/>
   </joint>
@@ -100,5 +100,5 @@
     <parent link="chassis_link"/>
     <child link="caster_wheel_link"/>
-    <origin xyz="${caster_x_offset} ${caster_y_offset} ${caster_z_offset}" rpy="0 0 0"/>
+    <origin xyz="${-caster_x_offset} ${caster_y_offset} ${caster_z_offset}" rpy="0 0 0"/>
     <axis xyz="0 0 1"/>
   </joint>
