Commit message: Tweaks to get robot working better

File: ora_description/description/robot_core.xacro (robot description, xacro)
@@ -8,6 +8,12 @@
   <xacro:include filename="inertia_macros.xacro"/>
   <!-- BASE LINK -->
-  <link name="base_link">
-  </link>
+  <link name="base_link"/>
+  <!-- BASE FOOTPRINT -->
+  <link name="base_footprint"/>
+  <joint name="base_footprint_join" type="fixed">
+    <parent link="base_link"/>
+    <child link="base_footprint"/>
+    <origin xyz="0 0 0" rpy="0 0 0"/>
+  </joint>
   <!-- CHASSIS LINK -->
   <joint name="chassis_joint" type="fixed">
@@ -100,5 +106,5 @@
     <visual>
       <geometry>
-        <sphere radius="${caster_radius}"/>
+        <sphere radius="${wheel_z_offset}"/>
       </geometry>
       <material name="black"/>
@@ -106,8 +112,8 @@
     <collision>
       <geometry>
-        <sphere radius="${caster_radius}"/>
+        <sphere radius="${wheel_z_offset}"/>
       </geometry>
     </collision>
-    <xacro:inertial_sphere mass="0.5" radius="${caster_radius}">
+    <xacro:inertial_sphere mass="0.5" radius="${wheel_z_offset}">
       <origin xyz="0 0 0" rpy="0 0 0"/>
     </xacro:inertial_sphere>

Commit message: flipped stuff around

File: ora_description/description/robot_core.xacro (robot description, xacro)
@@ -11,5 +11,5 @@
   <!-- BASE FOOTPRINT -->
   <link name="base_footprint"/>
-  <joint name="base_footprint_join" type="fixed">
+  <joint name="base_footprint_joint" type="fixed">
     <parent link="base_link"/>
     <child link="base_footprint"/>
@@ -20,5 +20,5 @@
     <parent link="base_link"/>
     <child link="chassis_link"/>
-    <origin xyz="-${wheel_x_offset} 0 0" rpy="0 0 0"/>
+    <origin xyz="${wheel_x_offset} 0 0" rpy="0 0 0"/>
   </joint>
   <link name="chassis_link">
@@ -48,6 +48,6 @@
     <parent link="base_link"/>
     <child link="left_wheel_link"/>
-    <origin xyz="0.0 ${wheel_y_offset} ${wheel_z_offset}" rpy="-${pi / 2} 0.0 0.0"/>
-    <axis xyz="0 0 1"/>
+    <origin xyz="${wheel_x_offset} ${wheel_y_offset} ${wheel_z_offset}" rpy="-${pi / 2} 0.0 0.0"/>
+    <axis xyz="0 0 -1"/>
   </joint>
   <link name="left_wheel_link">
@@ -74,6 +74,6 @@
     <parent link="base_link"/>
     <child link="right_wheel_link"/>
-    <origin xyz="0.0 -${wheel_y_offset} ${wheel_z_offset}" rpy="${pi / 2} 0.0 0.0"/>
-    <axis xyz="0 0 -1"/>
+    <origin xyz="${wheel_x_offset} -${wheel_y_offset} ${wheel_z_offset}" rpy="${pi / 2} 0.0 0.0"/>
+    <axis xyz="0 0 1"/>
   </joint>
   <link name="right_wheel_link">
@@ -100,5 +100,5 @@
     <parent link="chassis_link"/>
     <child link="caster_wheel_link"/>
-    <origin xyz="${caster_x_offset} ${caster_y_offset} ${caster_z_offset}" rpy="0 0 0"/>
+    <origin xyz="-${caster_x_offset} ${caster_y_offset} ${caster_z_offset}" rpy="0 0 0"/>
     <axis xyz="0 0 1"/>
   </joint>

Commit message: Fixed issues with footprint

File: ora_description/description/robot_core.xacro (robot description, xacro)
@@ -12,6 +12,6 @@
   <link name="base_footprint"/>
   <joint name="base_footprint_joint" type="fixed">
-    <parent link="base_link"/>
-    <child link="base_footprint"/>
+    <parent link="base_footprint"/>
+    <child link="base_link"/>
     <origin xyz="0 0 0" rpy="0 0 0"/>
   </joint>
